File: Cansat.kicad_sch (KiCad schematic)
At the start: 45 parts, among them J1 XT30_BATTERY, J10 Micro_SD_Card, J11 MAX17048_PLACEHOLDER, J12 BRIDGE_CAST_10, J13 PCB_A_SLOT_10, J14 BRIDGE_CAST_4, J15 PCB_B_SLOT_4, J2 BMP585_PLACEHOLDER, J3 BNO085_PLACEHOLDER, J4 CC1101_MODULE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

Commit message: Ready for PDR
Connections:
- net GPS_RX: now also U2.11 (GPIO18); no longer J12.6 (Pin_6)
- net GPS_TX: now also U2.10 (GPIO17); no longer J12.5 (Pin_5)
- net PPS: no longer J12.7 (Pin_7)
- net SCL_0: no longer J12.4 (Pin_4), J2.4 (Pin_4), J3.4 (Pin_4)
- net SDA_0: no longer J12.3 (Pin_3), J2.3 (Pin_3), J3.3 (Pin_3)
- net GPS_RX_BR: now reaches U4.18 (RX)
- net GPS_RX_BR: now also J12.6 (Pin_6); no longer U2.10 (GPIO17)
- net GPS_TX_BR: now reaches U4.17 (TX)
- net GPS_TX_BR: now also J12.5 (Pin_5); no longer U2.11 (GPIO18)
- net PPS_BR: now reaches U4.15 (PPS)
- net PPS_BR: now also J12.7 (Pin_7)
- new net SCL_0_BR: J12.4 (Pin_4), J2.4 (Pin_4), J3.4 (Pin_4)
- new net SDA_0_BR: J12.3 (Pin_3), J2.3 (Pin_3), J3.3 (Pin_3)
- no-connect marks 40 -> 38
Changed lines of the file:
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@@
 	)
 	(no_connect
-		(at 100.33 127)
-	)
-	(no_connect
 		(at 242.57 22.86)
 	)
@@
 	)
 	(no_connect
-		(at 204.47 114.3)
-	)
-	(no_connect
 		(at 45.72 160.02)
 	)
@@
 	(wire
 		(pts
-			(xy 97.79 121.92) (xy 97.79 120.65)
-		)
-		(stroke
-			(width 0)
-			(type default)
-		)
-	)
-	(wire
-		(pts
 			(xy 95.25 87.63) (xy 95.25 96.52)
 		)
@@
 	(wire
 		(pts
-			(xy 99.06 127) (xy 73.66 127)
-		)
-		(stroke
-			(width 0)
-			(type default)
-		)
-	)
-	(wire
-		(pts
 			(xy 96.52 85.09) (xy 102.87 85.09)
 		)
@@
 	(wire
 		(pts
-			(xy 97.79 120.65) (xy 85.09 120.65)
-		)
-		(stroke
-			(width 0)
-			(type default)
-		)
-	)
-	(wire
-		(pts
 			(xy 232.41 62.23) (xy 232.41 54.61)
 		)
@@
 	(wire
 		(pts
-			(xy 209.55 64.77) (xy 209.55 119.38)
-		)
-		(stroke
-			(width 0)
-			(type default)
-		)
-	)
-	(wire
-		(pts
 			(xy 33.02 157.48) (xy 45.72 157.48)
 		)
@@
 	(wire
 		(pts
-			(xy 85.09 128.27) (xy 72.39 128.27)
-		)
-		(stroke
-			(width 0)
-			(type default)
-		)
-	)
-	(wire
-		(pts
 			(xy 115.57 80.01) (xy 115.57 82.55)
 		)
@@
 	(wire
 		(pts
-			(xy 72.39 64.77) (xy 209.55 64.77)
-		)
-		(stroke
-			(width 0)
-			(type default)
-		)
-	)
-	(wire
-		(pts
 			(xy 266.7 48.26) (xy 271.78 48.26)
 		)
@@
 	(wire
 		(pts
-			(xy 73.66 127) (xy 73.66 68.58)
-		)
-		(stroke
-			(width 0)
-			(type default)
-		)
-	)
-	(wire
-		(pts
 			(xy 34.29 30.48) (xy 55.88 30.48)
 		)
@@
 	(wire
 		(pts
-			(xy 72.39 128.27) (xy 72.39 64.77)
-		)
-		(stroke
-			(width 0)
-			(type default)
-		)
-	)
-	(wire
-		(pts
 			(xy 135.89 148.59) (xy 135.89 149.86)
 		)
@@
 	(wire
 		(pts
-			(xy 99.06 119.38) (xy 99.06 127)
-		)
-		(stroke
-			(width 0)
-			(type default)
-		)
-	)
-	(wire
-		(pts
 			(xy 160.02 15.24) (xy 160.02 22.86)
 		)
@@
 	(wire
 		(pts
-			(xy 73.66 68.58) (xy 207.01 68.58)
-		)
-		(stroke
-			(width 0)
-			(type default)
-		)
-	)
-	(wire
-		(pts
 			(xy 228.6 115.57) (xy 250.19 115.57)
 		)
@@
 	(wire
 		(pts
-			(xy 85.09 120.65) (xy 85.09 128.27)
-		)
-		(stroke
-			(width 0)
-			(type default)
-		)
-	)
-	(wire
-		(pts
 			(xy 80.01 187.96) (xy 87.63 187.96)
 		)
@@
 	(wire
 		(pts
-			(xy 207.01 68.58) (xy 207.01 121.92)
-		)
-		(stroke
-			(width 0)
-			(type default)
-		)
-	)
-	(wire
-		(pts
 			(xy 100.33 99.06) (xy 95.25 99.06)
 		)
@@
 		)
 	)
-	(label "GPS_RX"
+	(label "GPS_RX_BR"
 		(at 166.37 151.13 0)
 		(effects
@@
 		)
 	)
-	(label "SDA_0"
+	(label "SDA_0_BR"
 		(at 166.37 143.51 0)
 		(effects
@@
 		)
 	)
+	(label "GPS_RX_BR"
+		(at 205.74 121.92 0)
+		(effects
+			(font
+				(size 1.27 1.27)
+			)
+			(justify left bottom)
+		)
+	)
 	(label "3V3"
 		(at 115.57 87.63 0)
@@
 		)
 	)
-	(label "SCL_0"
+	(label "SCL_0_BR"
 		(at 22.86 102.87 0)
 		(effects
@@
 		)
 	)
-	(label "SCL_0"
+	(label "SCL_0_BR"
 		(at 166.37 146.05 0)
 		(effects
@@
 		)
 	)
-	(label "SCL_0"
+	(label "SCL_0_BR"
 		(at 21.59 120.65 0)
 		(effects
@@
 		)
 	)
-	(label "SDA_0"
+	(label "SDA_0_BR"
 		(at 22.86 100.33 0)
 		(effects
@@
 		)
 	)
+	(label "GPS_RX"
+		(at 97.79 121.92 0)
+		(effects
+			(font
+				(size 1.27 1.27)
+			)
+			(justify left bottom)
+		)
+	)
 	(label "MOTOR1_PWM"
 		(at 74.93 110.49 0)
@@
 		)
 	)
+	(label "GPS_TX_BR"
+		(at 205.74 119.38 0)
+		(effects
+			(font
+				(size 1.27 1.27)
+			)
+			(justify left bottom)
+		)
+	)
 	(label "GND"
 		(at 24.13 115.57 0)
@@
 		)
 	)
-	(label "PPS"
+	(label "PPS_BR"
 		(at 166.37 153.67 0)
 		(effects
@@
 		)
 	)
-	(label "SDA_0"
+	(label "SDA_0_BR"
 		(at 21.59 118.11 0)
 		(effects
@@
 		)
 	)
-	(label "GPS_TX"
+	(label "GPS_TX_BR"
 		(at 166.37 148.59 0)
 		(effects
@@
 		)
 	)
+	(label "GPS_TX"
+		(at 99.06 119.38 0)
+		(effects
+			(font
+				(size 1.27 1.27)
+			)
+			(justify left bottom)
+		)
+	)
 	(label "SDA_0"
 		(at 228.6 156.21 180)
@@
 		(effects
 			(font
+				(size 1.27 1.27)
+			)
+			(justify left bottom)
+		)
+	)
+	(label "PPS_BR"
+		(at 204.47 114.3 0)
+		(effects
+			(font
