File: Cansat.kicad_pcb (KiCad board)
At the start: 2 copper layers, 40 parts, among them J1 XT30_BATTERY, J10 Micro_SD_Card, J11 MAX17048_PLACEHOLDER, J2 BMP585_PLACEHOLDER, J3 BNO085_PLACEHOLDER, J4 CC1101_MODULE, J5 BUZZ_CONN, J6 SERVO_OUTPUT, J7 5V_BEC, J8 ESC_4IN1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

Commit message: PDR Bridge Architecture: Generated custom courtyards and board outlines
Parts:
- added J12: BRIDGE_CAST_10, CanSat_Library:BRIDGE_CAST_10, F.Cu at (140.0, 119.5)
- added J13: PCB_A_SLOT_10, CanSat_Library:MAIN_EDGE_SLOT_10, F.Cu at (72.5, 127.0)
- added J14: BRIDGE_CAST_4, CanSat_Library:BRIDGE_CAST_4, F.Cu at (244.0, 121.5)
- added J15: PCB_B_SLOT_4, CanSat_Library:MAIN_EDGE_SLOT_4, F.Cu at (310.0, 122.5)
- added U6: AMS1117-3.3, Package_TO_SOT_SMD:SOT-223-3_TabPin2, F.Cu at (213.5, 97.0)
- J10: footprint Connector_PinSocket_2.54mm:PinSocket_1x08_P2.54mm_Vertical -> CanSat_Library:MicroSD_Breakout
- J11: footprint Connector_PinSocket_2.54mm:PinSocket_1x04_P2.54mm_Vertical -> CanSat_Library:MAX17048_Breakout
- J2: footprint Connector_PinSocket_2.54mm:PinSocket_1x04_P2.54mm_Vertical -> CanSat_Library:BMP585_Breakout
- J3: footprint Connector_PinSocket_2.54mm:PinSocket_1x04_P2.54mm_Vertical -> CanSat_Library:BNO085_Breakout
- J4: footprint Connector_PinSocket_2.54mm:PinSocket_1x08_P2.54mm_Vertical -> CanSat_Library:CC1101_Module
- J7: footprint Connector_PinSocket_2.54mm:PinSocket_1x04_P2.54mm_Vertical -> CanSat_Library:5V_BEC_Pololu
- J8: footprint Connector_PinSocket_2.54mm:PinSocket_1x08_P2.54mm_Vertical -> CanSat_Library:ESC_HAKRC_20A
- J9: footprint Connector_PinSocket_2.54mm:PinSocket_1x04_P2.54mm_Vertical -> CanSat_Library:SGP41_Breakout
- U3: footprint Connector_PinSocket_2.54mm:PinSocket_1x10_P2.54mm_Horizontal -> CanSat_Library:INA260_Breakout
- moved U4 180.7 mm to (286.7, 148.9)
- moved J11 147.5 mm to (35.5, 163.3)
- moved J4 147.2 mm to (310.0, 43.0)
- moved J10 125.5 mm to (303.0, 73.8)
- moved U1 116.3 mm to (38.0, 40.0)
- moved J3 103.2 mm to (105.0, 24.6)
- moved SW1 67.9 mm to (30.2, 108.5)
- moved U3 61.1 mm to (220.3, 60.5)
- moved J8 59.0 mm to (227.5, 108.0)
- moved U2 38.2 mm to (65.1, 25.7)
- moved J2 37.2 mm to (171.5, 145.5)
- moved R13 34.4 mm to (148.0, 150.9)
- moved R15 34.4 mm to (148.0, 159.0)
- moved R12 34.4 mm to (148.0, 146.8)
- moved R14 34.4 mm to (148.0, 154.9)
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Other:
- board outline added: 340 x 200 mm

Commit message: 3 PCB Design
Parts:
- moved J10 269.0 mm to (38.3, 122.0)
- moved SW1 253.7 mm to (283.8, 98.0)
- moved C5 248.6 mm to (306.5, 30.0)
- moved J11 229.4 mm to (241.0, 61.4)
- moved J4 228.8 mm to (98.0, 129.0)
- moved J1 169.6 mm to (288.0, 188.5)
- moved C2 164.9 mm to (301.5, 61.0)
- moved U4 158.0 mm to (148.2, 72.9)
- moved J6 157.3 mm to (253.0, 103.0)
- moved C1 148.2 mm to (29.0, 23.0)
- moved C4 138.2 mm to (57.0, 45.5)
- moved C7 136.2 mm to (34.8, 115.0)
- moved C3 124.0 mm to (57.0, 35.5)
- moved R8 122.9 mm to (57.0, 26.5)
- moved C6 122.9 mm to (24.0, 115.5)
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Other:
- board size 340 x 200 mm -> 1.8 x 32 mm

Commit message: Ready for PDR
Parts:
- moved C1 27.4 mm to (55.8, 17.0)
- moved U4 2.30 mm to (149.5, 71.0)
- moved J12 0.50 mm to (139.5, 119.5)
Connections:
- J12 pad 3: /SDA_0 -> /SDA_0_BR
- J12 pad 4: /SCL_0 -> /SCL_0_BR
- J12 pad 5: /GPS_TX -> /GPS_TX_BR
- J12 pad 6: /GPS_RX -> /GPS_RX_BR
- J12 pad 7: /PPS -> /PPS_BR
- J2 pad 3: /SDA_0 -> /SDA_0_BR
- J2 pad 4: /SCL_0 -> /SCL_0_BR
- J3 pad 3: /SDA_0 -> /SDA_0_BR
- J3 pad 4: /SCL_0 -> /SCL_0_BR
- U2 pad 10: Net-(U2-GPIO17) -> /GPS_TX
- U2 pad 11: Net-(U2-GPIO18) -> /GPS_RX
- U4 pad 15: unconnected-(U4-PPS-Pad15) -> /PPS_BR
- U4 pad 17: Net-(U2-GPIO18) -> /GPS_TX_BR
- U4 pad 18: Net-(U2-GPIO17) -> /GPS_RX_BR
Other:
- board size 1.8 x 32 mm -> 301 x 201 mm
Changed lines of the file:
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@@
 			(layers "*.Cu" "*.Mask")
 			(remove_unused_layers no)
-			(net "Net-(U2-GPIO17)")
+			(net "/GPS_TX")
 			(pinfunction "GPIO17_10")
 			(pintype "bidirectional")
@@
 			(layers "*.Cu" "*.Mask")
 			(remove_unused_layers no)
-			(net "Net-(U2-GPIO18)")
+			(net "/GPS_RX")
 			(pinfunction "GPIO18_11")
 			(pintype "bidirectional")
@@
 			(net "unconnected-(U2-GPIO3-Pad13)")
 			(pinfunction "GPIO3_13")
-			(pintype "bidirectional+no_connect")
+			(pintype "bidirectional")
 		)
 		(pad "14" thru_hole oval
@@
 	(footprint "CanSat_Library:BRIDGE_CAST_10"
 		(layer "F.Cu")
-		(at 140 119.5)
+		(at 139.5 119.5)
 		(property "Reference" "J12"
 			(at 2 0 90)
@@
 			(layers "*.Cu" "*.Mask")
 			(remove_unused_layers no)
-			(net "/SDA_0")
+			(net "/SDA_0_BR")
 			(pinfunction "Pin_3_3")
 			(pintype "passive")
@@
 			(layers "*.Cu" "*.Mask")
 			(remove_unused_layers no)
-			(net "/SCL_0")
+			(net "/SCL_0_BR")
 			(pinfunction "Pin_4_4")
 			(pintype "passive")
@@
 			(layers "*.Cu" "*.Mask")
 			(remove_unused_layers no)
-			(net "/GPS_TX")
+			(net "/GPS_TX_BR")
 			(pinfunction "Pin_5_5")
 			(pintype "passive")
@@
 			(layers "*.Cu" "*.Mask")
 			(remove_unused_layers no)
-			(net "/GPS_RX")
+			(net "/GPS_RX_BR")
 			(pinfunction "Pin_6_6")
 			(pintype "passive")
@@
 			(layers "*.Cu" "*.Mask")
 			(remove_unused_layers no)
-			(net "/PPS")
+			(net "/PPS_BR")
 			(pinfunction "Pin_7_7")
 			(pintype "passive")
@@
 			(layers "*.Cu" "*.Mask")
 			(remove_unused_layers no)
-			(net "/SDA_0")
+			(net "/SDA_0_BR")
 			(pinfunction "Pin_3_3")
 			(pintype "passive")
@@
 			(layers "*.Cu" "*.Mask")
 			(remove_unused_layers no)
-			(net "/SCL_0")
+			(net "/SCL_0_BR")
 			(pinfunction "Pin_4_4")
 			(pintype "passive")
@@
 	(footprint "CanSat_Library:Edgehax_NavIC"
 		(layer "F.Cu")
-		(at 148.23 72.92)
+		(at 149.5 71)
 		(property "Reference" "U4"
 			(at 25 -15 0)
@@
 			(layers "*.Cu" "*.Mask")
 			(remove_unused_layers no)
-			(net "unconnected-(U4-PPS-Pad15)")
+			(net "/PPS_BR")
 			(pinfunction "PPS_15")
-			(pintype "output+no_connect")
+			(pintype "output")
 		)
 		(pad "16" thru_hole circle
@@
 			(layers "*.Cu" "*.Mask")
 			(remove_unused_layers no)
-			(net "Net-(U2-GPIO18)")
+			(net "/GPS_TX_BR")
 			(pinfunction "TX_17")
 			(pintype "output")
@@
 			(layers "*.Cu" "*.Mask")
 			(remove_unused_layers no)
-			(net "Net-(U2-GPIO17)")
+			(net "/GPS_RX_BR")
 			(pinfunction "RX_18")
 			(pintype "input")
@@
 	(footprint "Capacitor_THT:C_Disc_D5.0mm_W2.5mm_P2.50mm"
 		(layer "F.Cu")
-		(at 29 23)
+		(at 55.75 17)
 		(descr "C, Disc series, Radial, pin pitch=2.50mm, diameter*width=5*2.5mm^2, Capacitor, http://cdn-reichelt.de/documents/datenblatt/B300/DS_KERKO_TC.pdf")
 		(tags "C Disc series Radial pin pitch 2.50mm diameter 5mm width 2.5mm Capacitor")
@@
 		(layer "F.Cu")
 		(at 38 40)
-		(descr "Digi XBee 3 Pro Through-Hole module, 20 pins, 2mm pitch, 22mm row spacing, UFL antenna")
-		(tags "XBee Digi RF Module TH UFL")
 		(property "Reference" "U1"
 			(at 0 -15 0)
@@
 		(duplicate_pad_numbers_are_jumpers no)
 		(fp_line
-			(start -12.7 -13.5)
-			(end 12.7 -13.5)
+			(start -12.19 -14.42)
+			(end -12.19 10.52)
 			(stroke
 				(width 0.12)
@@
 		)
 		(fp_line
-			(start -12.7 8.5)
-			(end -12.7 -13.5)
+			(start -12.19 10.52)
+			(end 12.19 10.52)
 			(stroke
 				(width 0.12)
@@
 		)
 		(fp_line
-			(start -7.5 13.5)
-			(end -12.7 8.5)
+			(start -7.5 -22.42)
+			(end -12.19 -14.42)
 			(stroke
 				(width 0.12)
@@
 		)
 		(fp_line
-			(start 7.5 13.5)
-			(end -7.5 13.5)
+			(start 7.5 -22.42)
+			(end -7.5 -22.42)
 			(stroke
 				(width 0.12)
@@
 		)
 		(fp_line
-			(start 12.7 -13.5)
-			(end 12.7 8.5)
+			(start 12.19 -14.42)
+			(end 7.5 -22.42)
 			(stroke
 				(width 0.12)
@@
 		)
 		(fp_line
-			(start 12.7 8.5)
-			(end 7.5 13.5)
+			(start 12.19 10.52)
+			(end 12.19 -14.42)
 			(stroke
 				(width 0.12)
@@
 		)
 		(fp_line
-			(start -13 -14)
-			(end 13 -14)
+			(start -12.5 -14.5)
+			(end -12.5 11)
+			(stroke
+				(width 0.05)
+				(type solid)
+			)
+			(layer "F.CrtYd")
+		)
+		(fp_line
+			(start -12.5 11)
+			(end 12.5 11)
+			(stroke
+				(width 0.05)
+				(type solid)
+			)
+			(layer "F.CrtYd")
+		)
+		(fp_line
+			(start -8 -23)
+			(end -12.5 -14.5)
 			(stroke
 				(width 0.05)
@@
 		)
 		(fp_line
-			(start -13 14)
-			(end -13 -14)
+			(start 8 -23)
+			(end -8 -23)
 			(stroke
 				(width 0.05)
@@
 		)
 		(fp_line
-			(start 13 -14)
-			(end 13 14)
+			(start 12.5 -14.5)
+			(end 8 -23)
 			(stroke
 				(width 0.05)
@@
 		)
 		(fp_line
-			(start 13 14)
-			(end -13 14)
+			(start 12.5 11)
+			(end 12.5 -14.5)
 			(stroke
 				(width 0.05)
@@
 		)
 		(fp_line
-			(start -12.7 -13.5)
-			(end 12.7 -13.5)
+			(start -12.19 -14.42)
+			(end -12.19 10.52)
 			(stroke
 				(width 0.1)
@@
 		)
 		(fp_line
-			(start -12.7 8.5)
-			(end -12.7 -13.5)
+			(start -12.19 10.52)
+			(end 12.19 10.52)
 			(stroke
 				(width 0.1)
@@
 		)
 		(fp_line
-			(start -7.5 13.5)
-			(end -12.7 8.5)
+			(start -7.5 -22.42)
+			(end -12.19 -14.42)
 			(stroke
 				(width 0.1)
@@
 		)
 		(fp_line
-			(start 7.5 13.5)
-			(end -7.5 13.5)
+			(start 7.5 -22.42)
+			(end -7.5 -22.42)
 			(stroke
 				(width 0.1)
@@
 		)
 		(fp_line
-			(start 12.7 -13.5)
-			(end 12.7 8.5)
+			(start 12.19 -14.42)
+			(end 7.5 -22.42)
 			(stroke
 				(width 0.1)
@@
 		)
 		(fp_line
-			(start 12.7 8.5)
-			(end 7.5 13.5)
+			(start 12.19 10.52)
+			(end 12.19 -14.42)
 			(stroke
 				(width 0.1)
@@
 		)
 		(pad "1" thru_hole rect
-			(at -11 -11.5)
+			(at -11 -9)
 			(size 1.5 1.5)
 			(drill 1)
@@
 		)
 		(pad "2" thru_hole circle
-			(at -11 -9.5)
+			(at -11 -7)
 			(size 1.5 1.5)
 			(drill 1)
@@
 		)
 		(pad "3" thru_hole circle
-			(at -11 -7.5)
+			(at -11 -5)
 			(size 1.5 1.5)
 			(drill 1)
@@
 		)
 		(pad "4" thru_hole circle
-			(at -11 -5.5)
+			(at -11 -3)
 			(size 1.5 1.5)
 			(drill 1)
@@
 		)
 		(pad "5" thru_hole circle
-			(at -11 -3.5)
+			(at -11 -1)
 			(size 1.5 1.5)
 			(drill 1)
@@
 		)
 		(pad "6" thru_hole circle
-			(at -11 -1.5)
+			(at -11 1)
 			(size 1.5 1.5)
 			(drill 1)
@@
 		)
 		(pad "7" thru_hole circle
-			(at -11 0.5)
+			(at -11 3)
 			(size 1.5 1.5)
 			(drill 1)
@@
 		)
 		(pad "8" thru_hole circle
-			(at -11 2.5)
+			(at -11 5)
 			(size 1.5 1.5)
 			(drill 1)
@@
 		)
 		(pad "9" thru_hole circle
-			(at -11 4.5)
+			(at -11 7)
 			(size 1.5 1.5)
 			(drill 1)
@@
 		)
 		(pad "10" thru_hole circle
-			(at -11 6.5)
+			(at -11 9)
 			(size 1.5 1.5)
 			(drill 1)
@@
 		)
 		(pad "11" thru_hole circle
-			(at 11 6.5)
+			(at 11 9)
 			(size 1.5 1.5)
 			(drill 1)
@@
 		)
 		(pad "12" thru_hole circle
-			(at 11 4.5)
+			(at 11 7)
 			(size 1.5 1.5)
 			(drill 1)
@@
 		)
 		(pad "13" thru_hole circle
-			(at 11 2.5)
+			(at 11 5)
 			(size 1.5 1.5)
 			(drill 1)
@@
 		)
 		(pad "14" thru_hole circle
-			(at 11 0.5)
+			(at 11 3)
 			(size 1.5 1.5)
 			(drill 1)
@@
 		)
 		(pad "15" thru_hole circle
-			(at 11 -1.5)
+			(at 11 1)
 			(size 1.5 1.5)
 			(drill 1)
@@
 		)
 		(pad "16" thru_hole circle
-			(at 11 -3.5)
+			(at 11 -1)
 			(size 1.5 1.5)
 			(drill 1)
@@
 		)
 		(pad "17" thru_hole circle
-			(at 11 -5.5)
+			(at 11 -3)
 			(size 1.5 1.5)
 			(drill 1)
@@
 		)
 		(pad "18" thru_hole circle
-			(at 11 -7.5)
+			(at 11 -5)
 			(size 1.5 1.5)
 			(drill 1)
@@
 		)
 		(pad "19" thru_hole circle
-			(at 11 -9.5)
+			(at 11 -7)
 			(size 1.5 1.5)
 			(drill 1)
@@
 		)
 		(pad "20" thru_hole circle
-			(at 11 -11.5)
+			(at 11 -9)
 			(size 1.5 1.5)
 			(drill 1)
@@
 			(layers "*.Cu" "*.Mask")
 			(remove_unused_layers no)
-			(net "/SDA_0")
+			(net "/SDA_0_BR")
 			(pinfunction "Pin_3_3")
 			(pintype "passive")
@@
 			(layers "*.Cu" "*.Mask")
 			(remove_unused_layers no)
-			(net "/SCL_0")
+			(net "/SCL_0_BR")
 			(pinfunction "Pin_4_4")
 			(pintype "passive")
@@
 		)
 		(fill no)
-		(layer "F.Cu")
+		(layer "Edge.Cuts")
 	)
 	(gr_rect
@@
 		)
 		(fill no)
-		(layer "F.Cu")
+		(layer "Edge.Cuts")
 	)
 	(gr_rect
@@
 		)
 		(fill no)
-		(layer "F.Cu")
-		(net "/BAT+")
+		(layer "Edge.Cuts")
 	)
 	(group ""

Commit message: Ready for PDR
Parts:
- moved R15 59.6 mm to (66.0, 202.5)
- moved R14 55.1 mm to (65.8, 194.0)
- moved C6 53.3 mm to (24.7, 168.8)
- moved C7 53.3 mm to (35.5, 168.3)
- moved J10 53.3 mm to (39.0, 175.3)
- moved J4 52.5 mm to (99.0, 181.5)
- moved R13 51.2 mm to (65.8, 186.0)
- moved J15 50.2 mm to (270.0, 115.0), turned to -90 degrees
- moved J13 49.0 mm to (70.0, 114.5), turned to -90 degrees
- moved R12 48.2 mm to (66.0, 179.0)
- moved R11 44.7 mm to (65.8, 172.0)
- moved SW1 37.2 mm to (301.8, 65.5)
- moved F1 37.1 mm to (228.4, 191.5)
- moved J5 35.7 mm to (258.5, 74.5)
- moved U5 35.1 mm to (172.5, 135.4)
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Other:
- outline, holes or cut-outs redrawn
- board text added: "100 mm"
- board text added: "200 mm"
- board text added: "66 mm"
