File: single_board/Cansat.kicad_pcb (KiCad board)
At the start: 2 copper layers, 1.8 x 32 mm, 45 parts, among them J1 XT30_BATTERY, J10 Micro_SD_Card, J11 MAX17048_PLACEHOLDER, J12 BRIDGE_CAST_10, J13 PCB_A_SLOT_10, J14 BRIDGE_CAST_4, J15 PCB_B_SLOT_4, J2 BMP585_PLACEHOLDER, J3 BNO085_PLACEHOLDER, J4 CC1101_MODULE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

Commit message: Add single_board variant; copy library files; WIP before footprint fix
Parts:
- moved C5 305.7 mm to (39.0, 178.0)
- moved SW1 249.3 mm to (35.0, 115.0)
- moved C2 191.7 mm to (111.5, 86.5)
- moved U6 191.3 mm to (69.7, 96.8)
- moved J6 189.4 mm to (77.0, 173.0)
- moved J5 189.0 mm to (60.5, 176.0)
- moved J11 188.7 mm to (101.5, 188.3)
- moved J1 185.4 mm to (103.0, 177.0)
- moved J7 181.2 mm to (103.8, 61.5)
- moved U3 177.9 mm to (95.5, 131.6)
- moved J8 177.6 mm to (106.5, 20.5)
- moved F1 158.1 mm to (88.5, 167.5)
- moved U4 141.7 mm to (27.7, 147.4)
- moved J2 130.7 mm to (37.1, 188.1)
- moved J9 130.7 mm to (70.5, 187.1)
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
Commit message: before patcher
Parts:
- removed J12: BRIDGE_CAST_10, CanSat_Library:BRIDGE_CAST_10
- removed J13: PCB_A_SLOT_10, CanSat_Library:MAIN_EDGE_SLOT_10
- removed J14: BRIDGE_CAST_4, CanSat_Library:BRIDGE_CAST_4
- removed J15: PCB_B_SLOT_4, CanSat_Library:MAIN_EDGE_SLOT_4
- moved J8 1.35 mm to (105.2, 20.5)
Other:
- board size 1.8 x 32 mm -> 100 x 200 mm

Commit message: Ready for PDR
Parts:
- moved C1 36.9 mm to (49.8, 53.5)
- moved R11 29.7 mm to (51.5, 46.5), turned to 180 degrees
- moved R12 21.4 mm to (51.5, 39.0), turned to 180 degrees
- moved R13 14.9 mm to (52.1, 33.4), turned to 180 degrees
- moved R14 7.11 mm to (52.1, 26.5), turned to 180 degrees
- moved U1 4.61 mm to (33.5, 41.0)
- moved R15 2.76 mm to (52.0, 20.0), turned to 180 degrees
Routing:
- net /VBAT_PROTECTED: track 0.00 -> 73.4 mm
- net /VBAT: track 0.00 -> 11.3 mm

Commit message: Ready for PDR
Parts:
- moved U5 99.7 mm to (24.5, 196.9)
- moved F1 34.4 mm to (56.4, 180.0)
- moved J9 32.1 mm to (102.0, 181.0)
- moved J11 31.0 mm to (100.5, 157.3)
- moved J1 28.1 mm to (105.5, 205.0)
- moved J6 27.5 mm to (77.0, 200.5)
- moved J5 26.8 mm to (62.5, 202.7)
- moved C5 24.6 mm to (36.6, 202.5)
- moved R5 22.6 mm to (45.0, 124.0), turned to 90 degrees
- moved R4 17.4 mm to (31.0, 124.0), turned to 90 degrees
- moved R1 16.6 mm to (38.0, 124.0), turned to 90 degrees
- moved J2 13.6 mm to (37.8, 174.5)
- moved SW1 9.28 mm to (32.8, 106.0)
- moved C2 8.39 mm to (113.0, 94.8), turned to 90 degrees
- moved R6 6.08 mm to (74.5, 94.5)
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Routing:
- net /VBAT_PROTECTED: track 73.4 -> 0.00 mm
- net /VBAT: track 11.3 -> 0.00 mm
Other:
- board text added: "100 mm"
- board text added: "200 mm"
